Commit message: Update: Added dragon hotend to urdf model and additional named pose states

File: catkin_ws/src/cram_v1/cram_description/urdf/common_colours.xacro (robot description, xacro)
@@ -10,3 +10,4 @@
 	<xacro:property name="color_black"    value="0.15 0.15 0.15 1.0" />
 	<xacro:property name="color_greyish"  value="0.75 0.75 0.75 1.0" />
+	<xacro:property name="color_red"  value="0.75 0.12 0.06 1.0" />
 </robot>

File: catkin_ws/src/cram_v1/cram_description/urdf/common_materials.xacro (robot description, xacro)
@@ -1,5 +1,5 @@
 <?xml version="1.0"?>
 <robot xmlns:xacro="http://ros.org/wiki/xacro">
-	<xacro:include filename="$(find widowx_arm_description)/urdf/common_colours.xacro"/>
+	<xacro:include filename="$(find cram_description)/urdf/common_colours.xacro"/>
 	<xacro:macro name="material_yellow">
 		<material name="">
@@ -27,3 +27,8 @@
 		</material>
 	</xacro:macro>
+	<xacro:macro name="material_red">
+		<material name="">
+			<color rgba="${color_red}"/>
+		</material>
+	</xacro:macro>
 </robot>

File: catkin_ws/src/cram_v1/cram_description/urdf/widowx.urdf.xacro (robot description, xacro)
@@ -10,5 +10,5 @@
             <origin xyz="0 0 0" rpy="0 0 0" />
             <geometry>
-               <mesh filename="package://widowx_arm_description/meshes/base_link.stl"/>
+               <mesh filename="package://cram_description/meshes/base_link.stl"/>
             </geometry>
             <xacro:material_black />
@@ -17,5 +17,5 @@
             <origin xyz="0 0 0" rpy="0 0 0" />
             <geometry>
-               <mesh filename="package://widowx_arm_description/meshes/base_link.stl"/>
+               <mesh filename="package://cram_description/meshes/base_link.stl"/>
             </geometry>
          </collision>
@@ -30,5 +30,5 @@
             <origin xyz="0 0 0" rpy="0 0 0" />
             <geometry>
-               <mesh filename="package://widowx_arm_description/meshes/shoulder_link.stl" />
+               <mesh filename="package://cram_description/meshes/shoulder_link.stl" />
             </geometry>
             <xacro:material_black />
@@ -37,5 +37,5 @@
             <origin xyz="0 0 0" rpy="0 0 0" />
             <geometry>
-               <mesh filename="package://widowx_arm_description/meshes/shoulder_link.stl"/>
+               <mesh filename="package://cram_description/meshes/shoulder_link.stl"/>
             </geometry>
          </collision>
@@ -51,5 +51,5 @@
             <!--origin xyz="0 0 0" rpy="0 0 0" /-->
             <geometry>
-               <mesh filename="package://widowx_arm_description/meshes/biceps_link.stl" />
+               <mesh filename="package://cram_description/meshes/biceps_link.stl" />
             </geometry>
             <xacro:material_black/>
@@ -58,5 +58,5 @@
             <origin xyz="${M_SCALE*48.25} 0 ${M_SCALE*140}" rpy="0 0 0" />
             <geometry>
-               <mesh filename="package://widowx_arm_description/meshes/biceps_link.stl" />
+               <mesh filename="package://cram_description/meshes/biceps_link.stl" />
             </geometry>
          </collision>
@@ -72,5 +72,5 @@
 			<!--origin xyz="0 0 0" rpy="0 0 0" /-->
             <geometry>
-               <mesh filename="package://widowx_arm_description/meshes/forearm_link.stl"/>
+               <mesh filename="package://cram_description/meshes/forearm_link.stl"/>
             </geometry>
            <xacro:material_black />
@@ -79,5 +79,5 @@
             <origin xyz="0 0 ${M_SCALE*142.03}" rpy="0 0 0" />
             <geometry>
-               <mesh filename="package://widowx_arm_description/meshes/forearm_link.stl"/>
+               <mesh filename="package://cram_description/meshes/forearm_link.stl"/>
             </geometry>
          </collision>
@@ -90,14 +90,34 @@
       <link name="${prefix}wrist_1_link">
          <visual>
-            <origin xyz="0 0 0" rpy="0 0 0" />
-            <geometry>
-               <mesh filename="package://widowx_arm_description/meshes/wrist_1_link.stl"/>
+            <origin xyz="0 0 0" rpy="-1.5707 0 0" />
+            <geometry>
+               <mesh scale="0.001 0.001 0.001" filename="package://cram_description/meshes/wrist_bracket.stl"/>
             </geometry>
             <xacro:material_black />
          </visual>
          <collision>
-            <origin xyz="0 0 0" rpy="0 0 0" />
-            <geometry>
-               <mesh filename="package://widowx_arm_description/meshes/wrist_1_link.stl"/>
+            <origin xyz="0 0 0" rpy="-1.5707 0 0" />
+            <geometry>
+               <mesh scale="0.001 0.001 0.001" filename="package://cram_description/meshes/wrist_bracket.stl"/>
+            </geometry>
+         </collision>
+         <inertial>
+            <origin xyz="0 0 0" rpy="0 0 0" />
+            <mass value="1" />
+            <inertia ixx="1.0" ixy="0.0" ixz="0.0" iyy="1.0" iyz="0.0" izz="1.0" />
+         </inertial>
+      </link>
+      <link name="${prefix}hotend">
+         <visual>
+            <origin xyz="0 0 ${M_SCALE*37}" rpy="0 0 -0.7854" />
+            <geometry>
+               <mesh scale="0.001 0.001 0.001" filename="package://cram_description/meshes/dragon_hotend.stl"/>
+            </geometry>
+            <xacro:material_red />
+         </visual>
+         <collision>
+            <origin xyz="0 0 ${M_SCALE*37}" rpy="0 0 -0.7854" />
+            <geometry>
+               <mesh scale="0.001 0.001 0.001" filename="package://cram_description/meshes/dragon_hotend.stl"/>
             </geometry>
          </collision>
@@ -142,4 +162,9 @@
          <axis xyz="0 1 0" />
          <limit lower="-1.745" upper="1.745" effort="0" velocity="8.168" />
+      </joint>
+      <joint name="${prefix}hotend" type="fixed">
+         <!--<insert_block name="origin" />-->
+         <parent link="${prefix}wrist_1_link" />
+         <child link="${prefix}hotend"/>
       </joint>
       <!--joint name="${prefix}joint_6" type="fixed">

File: catkin_ws/src/cram_v1/widowx_moveit/config/gazebo_widowx_arm.urdf (robot description, URDF)
Before this commit: robot widowx_arm, 6 links, 5 joints
Links:
- added link hotend, mass 1; collision mesh filename=package://cram_description/meshes/dragon_hotend.stl scale=0.001 0.001 0.001; visual mesh filename=package://cram_description/meshes/dragon_hotend.stl scale=0.001 0.001 0.001
- link arm_base_link: geometry collision mesh filename=package://cram_description/meshes/base_link.stl; visual mesh filename=package://cram_description/meshes/base_link.stl
- link biceps_link: geometry collision mesh filename=package://cram_description/meshes/biceps_link.stl; visual mesh filename=package://cram_description/meshes/biceps_link.stl
- link forearm_link: geometry collision mesh filename=package://cram_description/meshes/forearm_link.stl; visual mesh filename=package://cram_description/meshes/forearm_link.stl
- link shoulder_link: geometry collision mesh filename=package://cram_description/meshes/shoulder_link.stl; visual mesh filename=package://cram_description/meshes/shoulder_link.stl
- link wrist_1_link: geometry collision mesh filename=package://cram_description/meshes/wrist_bracket.stl scale=0.001 0.001 0.001; visual mesh filename=package://cram_description/meshes/wrist_bracket.stl scale=0.001 0.001 0.001
Joints:
- added joint hotend: type fixed, parent wrist_1_link, child hotend
- joint joint_1: limit lower=-2.617 upper=2.617 effort=0 velocity=0.785 -> lower=-2.617 upper=2.617 effort=0 velocity=7.016
- joint joint_2: limit lower=-1.571 upper=1.571 effort=0 velocity=1.571 -> lower=-1.571 upper=1.571 effort=0 velocity=5.760
- joint joint_3: limit lower=-1.571 upper=1.571 effort=0 velocity=1.571 -> lower=-1.571 upper=1.571 effort=0 velocity=5.760
- joint joint_4: limit lower=-1.745 upper=1.745 effort=0 velocity=1.571 -> lower=-1.745 upper=1.745 effort=0 velocity=8.168
