Commit message: Update: Added launch file for main cram ros module instead of using the moveit launch file. Modified cram urdf to more accurately mimic the current setup and updated the tfs.

File: catkin_ws/src/cram_v1/cram_description/robots/cram_v1_rig.urdf.xacro (robot description, xacro)
@@ -11,7 +11,7 @@
 	<link name="base">
 	<visual>
-	  <origin xyz="0 0 0.5" rpy="0 0 0"/>
+	  <origin xyz="0 0 0.02" rpy="0 0 0"/>
 	  <geometry>
-		<box size="1 2 1" />
+		<box size="0.31 0.935 0.04" />
 	  </geometry>
 	  <material name="White">
@@ -20,7 +20,7 @@
 	</visual>
 	<collision>
-	  <origin xyz="0 0 0.5" rpy="0 0 0"/>
+	  <origin xyz="0 0 0.02" rpy="0 0 0"/>
 	  <geometry>
-		<box size="1 1 1" />
+		<box size="0.31 0.935 0.04" />
 	  </geometry>
 	</collision>
@@ -28,7 +28,7 @@
 	<link name="buildplate">
 	<visual>
-	  <origin xyz="0 0 1" rpy="0 0 0"/>
+	  <origin xyz="0.15 0.15 0" rpy="0 0 0"/>
 	  <geometry>
-		<box size="0.3 0.3 0.01" />
+		<box size="0.3 0.3 0.004" />
 	  </geometry>
 	  <material name="Blue">
@@ -37,19 +37,20 @@
 	</visual>
 	<collision>
-	  <origin xyz="0 0 1" rpy="0 0 0"/>
+	  <origin xyz="0 0 0" rpy="0 0 0"/>
 	  <geometry>
-		<box size="0.3 0.3 0.01" />
+		<box size="0.3 0.3 0.004" />
 	  </geometry>
 	</collision>
 	</link>
 	<joint name="buildplate_joint" type="fixed">
+		<origin xyz="0.15 -0.15 0.04" rpy="0 0 1.5708"/>
 		<parent link="base"/>
 		<child link="buildplate"/>
 	</joint>
 	<!-- widowx arm with hotend -->
-	<xacro:widowx_arm arm_id="$(arg arm_id_1)" connected_to="base"  xyz="0 -0.245 1" rpy=" 0 0 1.5708 "/> />
+	<xacro:widowx_arm arm_id="$(arg arm_id_1)" connected_to="base"  xyz="0 -0.245 0.04" rpy=" 0 0 1.5708 "/> />
 	<xacro:hotend ns="$(arg arm_id_1)" rpy="0 0 0" connected_to="$(arg arm_id_1)_wrist_1_link"/>
 	<!-- widowxl arm with hotend -->
-	<xacro:widowx_arm arm_id="$(arg arm_id_2)" connected_to="base"  xyz="0 0.245 1" rpy="0 0 -1.5708"/> />
+	<xacro:widowx_arm arm_id="$(arg arm_id_2)" connected_to="base"  xyz="0 0.245 0.04" rpy="0 0 -1.5708"/> />
 	<xacro:hotend ns="$(arg arm_id_2)" rpy="0 0 0" connected_to="$(arg arm_id_2)_wrist_1_link"/>
 </robot>

Commit message: Update: Added demo python script for moveit commander

File: catkin_ws/src/cram_v1/cram_description/robots/cram_v1_rig.urdf.xacro (robot description, xacro)
@@ -6,5 +6,5 @@
   	<xacro:arg name="arm_id_2" default="widowx_2" />
 	<xacro:include filename="$(find cram_description )/urdf/widowx.urdf.xacro"/>
-<!--	<xacro:include filename="$(find cram_description )/urdf/widowxl.urdf.xacro"/>-->
+	<xacro:include filename="$(find cram_description )/urdf/widowxl.urdf.xacro"/>
 	<xacro:include filename="$(find cram_description )/urdf/hotend.urdf.xacro"/>
 	<!-- box shaped table as base for the 2 robot arms -->
@@ -37,5 +37,5 @@
 	</visual>
 	<collision>
-	  <origin xyz="0 0 0" rpy="0 0 0"/>
+	  <origin xyz="0.15 0.15 0" rpy="0 0 0"/>
 	  <geometry>
 		<box size="0.3 0.3 0.004" />
@@ -52,5 +52,5 @@
 	<xacro:hotend ns="$(arg arm_id_1)" rpy="0 0 0" connected_to="$(arg arm_id_1)_wrist_1_link"/>
 	<!-- widowxl arm with hotend -->
-	<xacro:widowx_arm arm_id="$(arg arm_id_2)" connected_to="base"  xyz="0 0.245 0.04" rpy="0 0 -1.5708"/> />
+	<xacro:widowxl_arm arm_id="$(arg arm_id_2)" connected_to="base"  xyz="0 0.245 0.04" rpy="0 0 -1.5708"/> />
 	<xacro:hotend ns="$(arg arm_id_2)" rpy="0 0 0" connected_to="$(arg arm_id_2)_wrist_1_link"/>
 </robot>

File: catkin_ws/src/cram_v1/cram_description/urdf/widowxl.urdf.xacro (robot description, xacro)
@@ -8,7 +8,7 @@
    <xacro:macro name="widowxl_arm" params="arm_id:='widowxl' arm_type:='widowxl' connected_to:='' xyz:='0 0 0' rpy:='0 0 0' description_pkg:='cram_description' ">
       <xacro:unless value="${not connected_to}">
-      <joint name="${arm_id}_joint_1" type="fixed">
+      <joint name="${arm_id}_joint_${connected_to}" type="fixed">
         <parent link="${connected_to}"/>
-        <child link="${arm_id}_link0"/>
+        <child link="${arm_id}_arm_base_link"/>
         <origin rpy="${rpy}" xyz="${xyz}"/>
       </joint>
@@ -118,5 +118,5 @@
       </link>
       <!-- joints -->
-      <joint name="joint_1" type="revolute">
+      <joint name="${arm_id}_joint_1" type="revolute">
          <origin xyz="0 0 ${M_SCALE*125}" rpy="0 0 0" />
          <parent link="${arm_id}_arm_base_link" />
@@ -125,5 +125,5 @@
          <limit lower="-2.617" upper="2.617" effort="0" velocity="7.016" />
       </joint>
-      <joint name="joint_2" type="revolute">
+      <joint name="${arm_id}_joint_2" type="revolute">
          <!--origin xyz="0.04825 0 0.14203" rpy="0 0 0" /-->
          <origin xyz="0 0 0" rpy="0 0 0" />
@@ -133,5 +133,5 @@
          <limit lower="-1.571" upper="1.571" effort="0" velocity="5.760" />
       </joint>
-      <joint name="joint_3" type="revolute">
+      <joint name="${arm_id}_joint_3" type="revolute">
          <origin xyz="${M_SCALE*48.25} 0 ${M_SCALE*142.03}" rpy="0 ${M_PI/2.0} 0" />
          <parent link="${arm_id}_biceps_link" />
@@ -140,5 +140,5 @@
          <limit lower="-1.571" upper="1.571" effort="0" velocity="5.760" />
       </joint>
-      <joint name="joint_4" type="revolute">
+      <joint name="${arm_id}_joint_4" type="revolute">
          <origin xyz="0 0 ${M_SCALE*142.03}" rpy="0 0 0" />
          <parent link="${arm_id}_forearm_link" />
@@ -148,35 +148,35 @@
       </joint>
    </xacro:macro>
-   <transmission name="tran1">
-    <type>transmission_interface/SimpleTransmission</type>
-    <joint name="joint_1"/>
-    <actuator name="motor1">
-      <hardwareInterface>hardware_interface/PositionJointInterface</hardwareInterface>
-      <mechanicalReduction>1</mechanicalReduction>
-    </actuator>
-  </transmission>
-   <transmission name="tran2">
-    <type>transmission_interface/SimpleTransmission</type>
-    <joint name="joint_2"/>
-    <actuator name="motor2">
-      <hardwareInterface>hardware_interface/PositionJointInterface</hardwareInterface>
-      <mechanicalReduction>1</mechanicalReduction>
-    </actuator>
-  </transmission>
-   <transmission name="tran3">
-    <type>transmission_interface/SimpleTransmission</type>
-    <joint name="joint_3"/>
-    <actuator name="motor3">
-      <hardwareInterface>hardware_interface/PositionJointInterface</hardwareInterface>
-      <mechanicalReduction>1</mechanicalReduction>
-    </actuator>
-  </transmission>
-   <transmission name="tran4">
-    <type>transmission_interface/SimpleTransmission</type>
-    <joint name="joint_4"/>
-    <actuator name="motor4">
-      <hardwareInterface>hardware_interface/PositionJointInterface</hardwareInterface>
-      <mechanicalReduction>1</mechanicalReduction>
-    </actuator>
-  </transmission>
+<!--   <transmission name="tran1">-->
+<!--    <type>transmission_interface/SimpleTransmission</type>-->
+<!--    <joint name="widowx_joint_1"/>-->
+<!--    <actuator name="motor1">-->
+<!--      <hardwareInterface>hardware_interface/PositionJointInterface</hardwareInterface>-->
+<!--      <mechanicalReduction>1</mechanicalReduction>-->
+<!--    </actuator>-->
+<!--  </transmission>-->
+<!--   <transmission name="tran2">-->
+<!--    <type>transmission_interface/SimpleTransmission</type>-->
+<!--    <joint name="widowx_joint_2"/>-->
+<!--    <actuator name="motor2">-->
+<!--      <hardwareInterface>hardware_interface/PositionJointInterface</hardwareInterface>-->
+<!--      <mechanicalReduction>1</mechanicalReduction>-->
+<!--    </actuator>-->
+<!--  </transmission>-->
+<!--   <transmission name="tran3">-->
+<!--    <type>transmission_interface/SimpleTransmission</type>-->
+<!--    <joint name="widowx_joint_3"/>-->
+<!--    <actuator name="motor3">-->
+<!--      <hardwareInterface>hardware_interface/PositionJointInterface</hardwareInterface>-->
+<!--      <mechanicalReduction>1</mechanicalReduction>-->
+<!--    </actuator>-->
+<!--  </transmission>-->
+<!--   <transmission name="tran4">-->
+<!--    <type>transmission_interface/SimpleTransmission</type>-->
+<!--    <joint name="widowx_joint_4"/>-->
+<!--    <actuator name="motor4">-->
+<!--      <hardwareInterface>hardware_interface/PositionJointInterface</hardwareInterface>-->
+<!--      <mechanicalReduction>1</mechanicalReduction>-->
+<!--    </actuator>-->
+<!--  </transmission>-->
 </robot>

Commit message: Milestone: Got a relatively reliable IK solver configurations for pose goal movements

File: catkin_ws/src/cram_v1/cram_description/robots/cram_v1_rig.urdf.xacro (robot description, xacro)
@@ -8,10 +8,10 @@
 	<xacro:include filename="$(find cram_description )/urdf/widowxl.urdf.xacro"/>
 	<xacro:include filename="$(find cram_description )/urdf/hotend.urdf.xacro"/>
-	<!-- box shaped table as base for the 2 robot arms -->
+	<!-- Base for the 2 robot arms -->
 	<link name="base">
 	<visual>
 	  <origin xyz="0 0 0.02" rpy="0 0 0"/>
 	  <geometry>
-		<box size="0.31 0.935 0.04" />
+		<box size="0.935 0.31 0.04" />
 	  </geometry>
 	  <material name="White">
@@ -22,5 +22,5 @@
 	  <origin xyz="0 0 0.02" rpy="0 0 0"/>
 	  <geometry>
-		<box size="0.31 0.935 0.04" />
+		<box size="0.935 0.31 0.04" />
 	  </geometry>
 	</collision>
@@ -44,13 +44,13 @@
 	</link>
 	<joint name="buildplate_joint" type="fixed">
-		<origin xyz="0.15 -0.15 0.04" rpy="0 0 1.5708"/>
+		<origin xyz="-0.15 -0.15 0.04" rpy="0 0 0"/>
 		<parent link="base"/>
 		<child link="buildplate"/>
 	</joint>
 	<!-- widowx arm with hotend -->
-	<xacro:widowx_arm arm_id="$(arg arm_id_1)" connected_to="base"  xyz="0 -0.245 0.04" rpy=" 0 0 1.5708 "/> />
+	<xacro:widowx_arm arm_id="$(arg arm_id_1)" connected_to="base"  xyz="-0.245 0  0.04" rpy=" 0 0 0 "/> />
 	<xacro:hotend ns="$(arg arm_id_1)" rpy="0 0 0" connected_to="$(arg arm_id_1)_wrist_1_link"/>
 	<!-- widowxl arm with hotend -->
-	<xacro:widowxl_arm arm_id="$(arg arm_id_2)" connected_to="base"  xyz="0 0.245 0.04" rpy="0 0 -1.5708"/> />
+	<xacro:widowxl_arm arm_id="$(arg arm_id_2)" connected_to="base"  xyz="0.245 0 0.04" rpy="0 0 3.14159"/> />
 	<xacro:hotend ns="$(arg arm_id_2)" rpy="0 0 0" connected_to="$(arg arm_id_2)_wrist_1_link"/>
 </robot>

File: catkin_ws/src/cram_v1/cram_description/urdf/widowx.urdf.xacro (robot description, xacro)
@@ -131,5 +131,5 @@
          <child link="${arm_id}_biceps_link" />
          <axis xyz="0 1 0" />
-         <limit lower="-1.571" upper="1.571" effort="0" velocity="5.760" />
+         <limit lower="-1.60" upper="1.60" effort="0" velocity="5.760" />
       </joint>
       <joint name="${arm_id}_joint_3" type="revolute">
@@ -145,5 +145,5 @@
          <child link="${arm_id}_wrist_1_link" />
          <axis xyz="0 1 0" />
-         <limit lower="-1.745" upper="1.745" effort="0" velocity="8.168" />
+         <limit lower="-1.60" upper="1.60" effort="0" velocity="8.168" />
       </joint>
    </xacro:macro>

File: catkin_ws/src/cram_v1/cram_description/urdf/widowxl.urdf.xacro (robot description, xacro)
@@ -145,5 +145,5 @@
          <child link="${arm_id}_wrist_1_link" />
          <axis xyz="0 1 0" />
-         <limit lower="-1.745" upper="1.745" effort="0" velocity="8.168" />
+         <limit lower="-1.60" upper="1.60" effort="0" velocity="8.168" />
       </joint>
    </xacro:macro>

Commit message: Update: modified xacro files to include wrist joint

File: catkin_ws/src/cram_v1/cram_description/robots/cram_v1_rig.urdf.xacro (robot description, xacro)
@@ -5,4 +5,6 @@
 	<xacro:arg name="arm_id_1" default="widowx_1" />
   	<xacro:arg name="arm_id_2" default="widowx_2" />
+	<xacro:property name="M_SCALE" value="0.001"/>
+	<xacro:property name="M_PI" value="3.14159"/>
 	<xacro:include filename="$(find cram_description )/urdf/widowx.urdf.xacro"/>
 	<xacro:include filename="$(find cram_description )/urdf/widowxl.urdf.xacro"/>
@@ -49,8 +51,24 @@
 	</joint>
 	<!-- widowx arm with hotend -->
-	<xacro:widowx_arm arm_id="$(arg arm_id_1)" connected_to="base"  xyz="-0.245 0  0.04" rpy=" 0 0 0 "/> />
-	<xacro:hotend ns="$(arg arm_id_1)" rpy="0 0 0" connected_to="$(arg arm_id_1)_wrist_1_link"/>
+	<xacro:widowx_arm arm_id="$(arg arm_id_1)" connected_to="base"  xyz="-0.245 0  0.04" rpy=" 0 0 0 "/>
+<!--	<xacro:hotend ns="$(arg arm_id_1)" rpy="0 0 0" connected_to="$(arg arm_id_1)_wrist_1_link"/>-->
+	<xacro:hotend ns="$(arg arm_id_1)"/>
+	<joint name="$(arg arm_id_1)_joint_5" type="revolute">
+         <origin xyz="0 0 ${M_SCALE*71.5}" rpy="0 0 0" />
+         <parent link="$(arg arm_id_1)_wrist_1_link" />
+         <child link="$(arg arm_id_1)_hotend" />
+         <axis xyz="0 0 1" />
+         <limit lower="-2.617" upper="2.617" effort="0" velocity="1.571" />
+	</joint>
 	<!-- widowxl arm with hotend -->
-	<xacro:widowxl_arm arm_id="$(arg arm_id_2)" connected_to="base"  xyz="0.245 0 0.04" rpy="0 0 3.14159"/> />
-	<xacro:hotend ns="$(arg arm_id_2)" rpy="0 0 0" connected_to="$(arg arm_id_2)_wrist_1_link"/>
+	<xacro:widowxl_arm arm_id="$(arg arm_id_2)" connected_to="base"  xyz="0.245 0 0.04" rpy="0 0 3.14159"/>
+<!--	<xacro:hotend ns="$(arg arm_id_2)" rpy="0 0 0" connected_to="$(arg arm_id_2)_wrist_1_link"/>-->
+	<xacro:hotend ns="$(arg arm_id_2)" />
+		<joint name="$(arg arm_id_2)_joint_5" type="revolute">
+         <origin xyz="0 0 ${M_SCALE*71.5}" rpy="0 0 0" />
+         <parent link="$(arg arm_id_2)_wrist_1_link" />
+         <child link="$(arg arm_id_2)_hotend" />
+         <axis xyz="0 0 1" />
+         <limit lower="-2.617" upper="2.617" effort="0" velocity="1.571" />
+	</joint>
 </robot>

File: catkin_ws/src/cram_v1/cram_description/urdf/widowx.urdf.xacro (robot description, xacro)
@@ -101,5 +101,5 @@
             <origin xyz="0 0 0" rpy="-1.5707 0 0" />
             <geometry>
-               <mesh scale="0.001 0.001 0.001" filename="package://${description_pkg}/meshes/widowx/wrist_bracket.stl"/>
+               <mesh scale="0.001 0.001 0.001" filename="package://${description_pkg}/meshes/widowx/wrist_1_link.stl/>
             </geometry>
             <xacro:material_black />
@@ -108,13 +108,33 @@
             <origin xyz="0 0 0" rpy="-1.5707 0 0" />
             <geometry>
-               <mesh scale="0.001 0.001 0.001" filename="package://${description_pkg}/meshes/widowx/wrist_bracket.stl"/>
-            </geometry>
-         </collision>
-         <inertial>
-            <origin xyz="0 0 0" rpy="0 0 0" />
-            <mass value="1" />
-            <inertia ixx="1.0" ixy="0.0" ixz="0.0" iyy="1.0" iyz="0.0" izz="1.0" />
-         </inertial>
-      </link>
+               <mesh scale="0.001 0.001 0.001" filename="package://${description_pkg}/meshes/widowx/wrist_1_link.stl"/>
+            </geometry>
+         </collision>
+         <inertial>
+            <origin xyz="0 0 0" rpy="0 0 0" />
+            <mass value="1" />
+            <inertia ixx="1.0" ixy="0.0" ixz="0.0" iyy="1.0" iyz="0.0" izz="1.0" />
+         </inertial>
+      </link>
+<!--           <link name="${prefix}wrist_1_link">-->
+<!--         <visual>-->
+<!--            <origin xyz="0 0 ${M_SCALE*43}" rpy="0 0 0" />-->
+<!--            <geometry>-->
+<!--               <mesh scale="0.001 0.001 0.001" filename="package://${description_pkg}/meshes/widowx/wrist_1_link.stl"/>-->
+<!--            </geometry>-->
+<!--            <xacro:material_black />-->
+<!--         </visual>-->
+<!--         <collision>-->
+<!--            <origin xyz="0 0 0" rpy="0 0 0" />-->
+<!--            <geometry>-->
+<!--               <mesh scale="0.001 0.001 0.001" filename="package://${description_pkg}/meshes/widowx/wrist_1_link.stl"/>-->
+<!--            </geometry>-->
+<!--         </collision>-->
+<!--         <inertial>-->
+<!--            <origin xyz="0 0 0" rpy="0 0 0" />-->
+<!--            <mass value="1" />-->
+<!--            <inertia ixx="1.0" ixy="0.0" ixz="0.0" iyy="1.0" iyz="0.0" izz="1.0" />-->
+<!--         </inertial>-->
+<!--      </link>-->
       <!-- joints -->
       <joint name="${arm_id}_joint_1" type="revolute">

Commit message: Update: Modified urdf files to include additional degree of freedom at hotend

File: catkin_ws/src/cram_v1/cram_description/robots/cram_v1_rig.urdf.xacro (robot description, xacro)
@@ -52,23 +52,7 @@
 	<!-- widowx arm with hotend -->
 	<xacro:widowx_arm arm_id="$(arg arm_id_1)" connected_to="base"  xyz="-0.245 0  0.04" rpy=" 0 0 0 "/>
-<!--	<xacro:hotend ns="$(arg arm_id_1)" rpy="0 0 0" connected_to="$(arg arm_id_1)_wrist_1_link"/>-->
-	<xacro:hotend ns="$(arg arm_id_1)"/>
-	<joint name="$(arg arm_id_1)_joint_5" type="revolute">
-         <origin xyz="0 0 ${M_SCALE*71.5}" rpy="0 0 0" />
-         <parent link="$(arg arm_id_1)_wrist_1_link" />
-         <child link="$(arg arm_id_1)_hotend" />
-         <axis xyz="0 0 1" />
-         <limit lower="-2.617" upper="2.617" effort="0" velocity="1.571" />
-	</joint>
+	<xacro:hotend ns="$(arg arm_id_1)"  connected_to="$(arg arm_id_1)_wrist_1_link" xyz="0 0 ${M_SCALE*36.5}" rpy="0 0 ${-M_PI/4}" />
 	<!-- widowxl arm with hotend -->
-	<xacro:widowxl_arm arm_id="$(arg arm_id_2)" connected_to="base"  xyz="0.245 0 0.04" rpy="0 0 3.14159"/>
-<!--	<xacro:hotend ns="$(arg arm_id_2)" rpy="0 0 0" connected_to="$(arg arm_id_2)_wrist_1_link"/>-->
-	<xacro:hotend ns="$(arg arm_id_2)" />
-		<joint name="$(arg arm_id_2)_joint_5" type="revolute">
-         <origin xyz="0 0 ${M_SCALE*71.5}" rpy="0 0 0" />
-         <parent link="$(arg arm_id_2)_wrist_1_link" />
-         <child link="$(arg arm_id_2)_hotend" />
-         <axis xyz="0 0 1" />
-         <limit lower="-2.617" upper="2.617" effort="0" velocity="1.571" />
-	</joint>
+	<xacro:widowxl_arm arm_id="$(arg arm_id_2)" connected_to="base"  xyz="0.245 0 0.04" rpy="0 0 ${M_PI}"/>
+	<xacro:hotend ns="$(arg arm_id_2)" connected_to="$(arg arm_id_2)_wrist_1_link" xyz="0 0 ${M_SCALE*36.5}" rpy="0 0 ${-M_PI/4}" />
 </robot>

File: catkin_ws/src/cram_v1/cram_description/urdf/hotend.urdf.xacro (robot description, xacro)
@@ -3,9 +3,12 @@
  widowx xacro from https://github.com/RobotnikAutomation/widowx_arm -->
 <robot xmlns:xacro="http://www.ros.org/wiki/xacro" name="hotend">
-  <xacro:macro name="hotend" params="connected_to:='' ns:='' rpy:='0 0 0' xyz:='0 0 0' description_pkg:='cram_description' ">
+  <xacro:macro name="hotend" params="connected_to:='' ns:='' rpy:='' xyz:='' description_pkg:='cram_description' ">
     <xacro:unless value="${connected_to == ''}">
-      <joint name="${ns}_hotend_joint" type="fixed">
+      <joint name="${ns}_hotend_joint" type="revolute">
+<!--        <origin xyz="0 0 ${M_SCALE*71.5}" rpy="0 0 0" />-->
         <parent link="${connected_to}"/>
         <child link="${ns}_hotend"/>
+        <axis xyz="0 0 1" />
+        <limit lower="-2.617" upper="2.617" effort="0" velocity="1.571" />
         <origin xyz="${xyz}" rpy="${rpy}"/>
       </joint>
@@ -13,5 +16,5 @@
     <link name="${ns}_hotend">
          <visual>
-            <origin xyz="0 0 ${M_SCALE*37}" rpy="0 0 -0.7854" />
+            <origin xyz="${xyz}" rpy="${rpy}"/>
             <geometry>
                <mesh scale="0.001 0.001 0.001" filename="package://${description_pkg}/meshes/hotend/dragon_hotend.stl"/>
@@ -20,5 +23,5 @@
          </visual>
          <collision>
-            <origin xyz="0 0 ${M_SCALE*37}" rpy="0 0 -0.7854" />
+            <origin xyz="${xyz}" rpy="${rpy}" />
             <geometry>
                <mesh scale="0.001 0.001 0.001" filename="package://${description_pkg}/meshes/hotend/dragon_hotend.stl"/>
@@ -33,2 +36,8 @@
   </xacro:macro>
 </robot>
+<!--      <joint name="${prefix}joint_5" type="revolute">-->
+<!--         <origin xyz="0 0 ${M_SCALE*71.5}" rpy="0 0 0" />-->
+<!--         <parent link="${prefix}wrist_1_link" />-->
+<!--         <child link="${prefix}wrist_2_link" />-->
+<!--         <axis xyz="0 0 1" />-->
+<!--         <limit lower="-2.617" upper="2.617" effort="0" velocity="1.571" />-->

File: catkin_ws/src/cram_v1/cram_description/urdf/widowx.urdf.xacro (robot description, xacro)
@@ -99,14 +99,14 @@
       <link name="${arm_id}_wrist_1_link">
          <visual>
-            <origin xyz="0 0 0" rpy="-1.5707 0 0" />
+            <origin xyz="0 0 0" rpy="0 0 -3.141" />-->
             <geometry>
-               <mesh scale="0.001 0.001 0.001" filename="package://${description_pkg}/meshes/widowx/wrist_1_link.stl/>
+               <mesh filename="package://${description_pkg}/meshes/widowx/wrist_1_link.stl"/>
             </geometry>
             <xacro:material_black />
          </visual>
          <collision>
-            <origin xyz="0 0 0" rpy="-1.5707 0 0" />
+            <origin xyz="0 0 0" rpy="0 0 -3.141" />
             <geometry>
-               <mesh scale="0.001 0.001 0.001" filename="package://${description_pkg}/meshes/widowx/wrist_1_link.stl"/>
+               <mesh filename="package://${description_pkg}/meshes/widowx/wrist_1_link.stl"/>
             </geometry>
          </collision>
@@ -117,24 +117,4 @@
          </inertial>
       </link>
-<!--           <link name="${prefix}wrist_1_link">-->
-<!--         <visual>-->
-<!--            <origin xyz="0 0 ${M_SCALE*43}" rpy="0 0 0" />-->
-<!--            <geometry>-->
-<!--               <mesh scale="0.001 0.001 0.001" filename="package://${description_pkg}/meshes/widowx/wrist_1_link.stl"/>-->
-<!--            </geometry>-->
-<!--            <xacro:material_black />-->
-<!--         </visual>-->
-<!--         <collision>-->
-<!--            <origin xyz="0 0 0" rpy="0 0 0" />-->
-<!--            <geometry>-->
-<!--               <mesh scale="0.001 0.001 0.001" filename="package://${description_pkg}/meshes/widowx/wrist_1_link.stl"/>-->
-<!--            </geometry>-->
-<!--         </collision>-->
-<!--         <inertial>-->
-<!--            <origin xyz="0 0 0" rpy="0 0 0" />-->
-<!--            <mass value="1" />-->
-<!--            <inertia ixx="1.0" ixy="0.0" ixz="0.0" iyy="1.0" iyz="0.0" izz="1.0" />-->
-<!--         </inertial>-->
-<!--      </link>-->
       <!-- joints -->
       <joint name="${arm_id}_joint_1" type="revolute">

File: catkin_ws/src/cram_v1/cram_description/urdf/widowxl.urdf.xacro (robot description, xacro)
@@ -99,14 +99,14 @@
       <link name="${arm_id}_wrist_1_link">
          <visual>
-            <origin xyz="0 0 0" rpy="-1.5707 0 0" />
+            <origin xyz="0 0 0" rpy="0 0 -3.141" />-->
             <geometry>
-               <mesh scale="0.001 0.001 0.001" filename="package://${description_pkg}/meshes/widowxl/wrist_bracket.stl"/>
+               <mesh filename="package://${description_pkg}/meshes/widowx/wrist_1_link.stl"/>
             </geometry>
             <xacro:material_black />
          </visual>
          <collision>
-            <origin xyz="0 0 0" rpy="-1.5707 0 0" />
+            <origin xyz="0 0 0" rpy="0 0 -3.141" />
             <geometry>
-               <mesh scale="0.001 0.001 0.001" filename="package://${description_pkg}/meshes/widowxl/wrist_bracket.stl"/>
+               <mesh filename="package://${description_pkg}/meshes/widowx/wrist_1_link.stl"/>
             </geometry>
          </collision>
